Commit message: 修改：     launch/orchard/AprilTag/L_tags.yaml 	新文件：   launch/orchard/AprilTag/L_tags_2.yaml 	修改：     launch/orchard/Camera_setup/HML.xacro

File: launch/orchard/Camera_setup/HML.xacro (robot description, xacro)
@@ -44,18 +44,23 @@
     </visual>
   </link>
+<!--
+  origin是 child 相对于 parent 的初始位置和方向
+  child 坐标系下的点，可以通过左乘的方式来变换到 parent 下
+  箭头由 child 指向 parent
+ -->
   <joint name="base_to_cameraH_tf" type="fixed">
     <parent link="/M_camera_base" />
     <child link="/H_camera_base" />
-<origin xyz="0.089114 0.002120 0.203885" rpy="3.131217 -3.028817 3.141392" />
+<origin xyz="-0.105839 0.011434 0.544613" rpy="3.129876 -3.139335 -3.127100" />
   </joint>
   <joint name="base_to_cameraM_tf" type="fixed">
     <parent link="/L_camera_base" />
     <child link="/M_camera_base" />
-<origin xyz="0.201731 0.006230 0.235697" rpy="3.137621 2.883057 3.137947" />
+<origin xyz="-0.200750 -0.000253 0.534473" rpy="3.140458 -2.933073 3.140895" />
   </joint>
   <joint name="base_to_cameraL_tf" type="fixed">
     <parent link="/base_frame" />
     <child link="/L_camera_base" />
-    <origin xyz="0 0 0.300" rpy="3.1357474659609688 -0.7177994043808186 0" />
+<origin xyz=" 0 0 0.2 " rpy="3.12277 2.77351  3.1396" />
   </joint>
 </robot>
